Commit message: support navigation

File: src/g1_description/urdf/g1_comp.urdf (robot description, URDF)
Before this commit: robot g1_comp, 34 links, 33 joints
Links:
- removed link imu_in_pelvis
- removed link pelvis
- removed link pelvis_contour_link
- added link base_link, mass 3.813; visual mesh filename=package://g1_description/meshes/base_link.STL
- added link base_link_contour_link, mass 0.001; collision mesh filename=package://g1_description/meshes/base_link_contour_link.STL; visual mesh filename=package://g1_description/meshes/base_link_contour_link.STL
- added link imu_in_base_link
Joints:
- removed joint imu_in_pelvis_joint
- removed joint pelvis_contour_joint
- added joint base_link_contour_joint: type fixed, parent base_link, child base_link_contour_link
- added joint imu_in_base_link_joint: type fixed, parent base_link, child imu_in_base_link, origin xyz=0.04525 0 -0.08339 rpy=0 0 0
- joint left_hip_pitch_joint: parent pelvis -> base_link
- joint right_hip_pitch_joint: parent pelvis -> base_link
- joint waist_yaw_joint: parent pelvis -> base_link

Commit message: Back link name

File: src/g1_description/urdf/g1_comp.urdf (robot description, URDF)
Before this commit: robot g1_comp, 34 links, 33 joints
Links:
- removed link base_link
- removed link base_link_contour_link
- removed link imu_in_base_link
- added link imu_in_pelvis
- added link pelvis, mass 3.813; visual mesh filename=package://g1_description/meshes/pelvis.STL
- added link pelvis_contour_link, mass 0.001; collision mesh filename=package://g1_description/meshes/pelvis_contour_link.STL; visual mesh filename=package://g1_description/meshes/pelvis_contour_link.STL
Joints:
- removed joint base_link_contour_joint
- removed joint imu_in_base_link_joint
- added joint imu_in_pelvis_joint: type fixed, parent pelvis, child imu_in_pelvis, origin xyz=0.04525 0 -0.08339 rpy=0 0 0
- added joint pelvis_contour_joint: type fixed, parent pelvis, child pelvis_contour_link
- joint left_hip_pitch_joint: parent base_link -> pelvis
- joint right_hip_pitch_joint: parent base_link -> pelvis
- joint waist_yaw_joint: parent base_link -> pelvis

Commit message: change mid360 angle

File: src/g1_description/urdf/g1_comp.urdf (robot description, URDF)
Before this commit: robot g1_comp, 34 links, 33 joints
Joints:
- joint mid360_joint: origin xyz=0.0002835 0.00003 0.41618 rpy=3.14 0.04014257279586953 0 -> xyz=0.0002835 0.00003 0.41618 rpy=0 0.04014257279586953 0
