Commit message: Fix Lidar pose

File: src/g1_description/urdf/g1_23dof.urdf (robot description, URDF)
Before this commit: robot g1_23dof, 33 links, 32 joints
Joints:
- joint mid360_joint: origin xyz=0.0002835 0.00003 0.40618 rpy=0 0.04014257279586953 0 -> xyz=0.0002835 0.00003 0.40618 rpy=3.14 0.04014257279586953 0

File: src/g1_description/urdf/g1_comp.urdf (robot description, URDF)
Before this commit: robot g1_comp, 34 links, 33 joints
Joints:
- joint mid360_joint: origin xyz=0.0002835 0.00003 0.41618 rpy=0 0.04014257279586953 0 -> xyz=0.0002835 0.00003 0.41618 rpy=3.14 0.04014257279586953 0

Commit message: Add livx_frame

File: src/g1_description/urdf/g1_23dof.urdf (robot description, URDF)
Before this commit: robot g1_23dof, 33 links, 32 joints
Links:
- added link base_link
- added link livox_frame
Joints:
- added joint base_link_to_pelvis: type fixed, parent base_link, child pelvis, origin xyz=0 0 0 rpy=0 0 0
- added joint livox_joint: type fixed, parent torso_link, child livox_frame, origin xyz=0.0002835 0.00003 0.40618 rpy=3.14 0.04014257279586953 0

File: src/g1_description/urdf/g1_comp.urdf (robot description, URDF)
Before this commit: robot g1_comp, 35 links, 34 joints
Links:
- added link livox_frame
Joints:
- added joint livox_joint: type fixed, parent torso_link, child livox_frame, origin xyz=0.0002835 0.00003 0.40618 rpy=3.14 0.04014257279586953 0
