Commit message: D455 による Navigation 最適化 by sakamaki

File: src/g1_description/urdf/erasers_g1.urdf (robot description, URDF)
Before this commit: robot g1_comp, 38 links, 37 joints
Joints:
- joint d455_joint: origin xyz=0.0295 0 0.013 rpy=0 0 0 -> xyz=0.0295 0 0.013 rpy=0 0.1 0

Commit message: G1 頭部カメラを最適化

File: src/g1_description/urdf/erasers_g1.urdf (robot description, URDF)
Before this commit: robot g1_comp, 38 links, 37 joints
Joints:
- joint d455_joint: limit lower=-0.3491 upper=1.5708 effort=0 velocity=0 -> lower=-1.57 upper=0.8 effort=0 velocity=0
- joint xl330_joint: limit lower=-0.8727 upper=0.8727 effort=0 velocity=0 -> lower=-0.7 upper=0.7 effort=0 velocity=0

File: src/g1_description/urdf/g1_comp.urdf (robot description, URDF)
Before this commit: robot g1_comp, 36 links, 35 joints
Joints:
- joint d455_joint: limit lower=-0.3491 upper=1.5708 effort=0 velocity=0 -> lower=-1.57 upper=1.0 effort=0 velocity=0
- joint xl330_joint: limit lower=-0.8727 upper=0.8727 effort=0 velocity=0 -> lower=-0.7 upper=0.7 effort=0 velocity=0
