Commit message: update ver2.0

File: src/erasers_g1_description/urdf/erasers_g1.urdf (robot description, URDF)
Before this commit: robot g1_comp, 38 links, 37 joints
Joints:
- joint left_amazing_hand_joint: origin xyz=0.16 0 0 rpy=0 0 0 -> xyz=0.16 0 0 rpy=3.141592653589793 0 0

File: src/erasers_g1_description/urdf/erasers_g1.urdf.xacro (robot description, xacro)
@@ -5,5 +5,8 @@
   <xacro:include filename="$(find erasers_g1_description)/urdf/g1_comp.urdf" />
   <!-- EE -->
-  <xacro:property name="ee_origin">
+  <xacro:property name="left_ee_origin">
+    <origin xyz="0.16 0 0" rpy="${pi} 0 0"/>
+  </xacro:property>
+  <xacro:property name="right_ee_origin">
     <origin xyz="0.16 0 0" rpy="0 0 0"/>
   </xacro:property>
@@ -12,5 +15,5 @@
     <parent link="left_wrist_roll_rubber_hand"/>
     <child link="left_amazing_hand"/>
-    <xacro:insert_block name="ee_origin"/>
+    <xacro:insert_block name="left_ee_origin"/>
   </joint>
   <link name="right_amazing_hand"/>
@@ -18,5 +21,5 @@
     <parent link="right_wrist_roll_rubber_hand"/>
     <child link="right_amazing_hand"/>
-    <xacro:insert_block name="ee_origin"/>
+    <xacro:insert_block name="right_ee_origin"/>
   </joint>
   <!-- ros2_control configuration -->
